Commit message: configuration files corrections
added corrections to robot urdf files (my_robot.xacro, my_robot.gazebo and mapping.launch files. most of them are documented on Q&A section of udacity.

File: catkin_ws/src/my_robot/urdf/my_robot.xacro (robot description, xacro)
@@ -141,4 +141,7 @@
     </visual>
   </link>
+  <!-- RGB-D Camera -->
+  <link name="camera_link_optical">
+  </link>
   <!-- joints -->
   <joint name="robot_footprint_joint" type="fixed">
@@ -176,4 +179,9 @@
     <axis xyz="0 1 0" rpy="0 0 0"/>
   </joint>
+  <joint name="camera_optical_joint" type="fixed">
+    <origin xyz="0 0 0" rpy="-1.5707 0 -1.5707"/>
+    <parent link="camera_link"/>
+    <child link="camera_link_optical"/>
+  </joint>
   <!-- colors -->
   <gazebo reference="left_wheel">

Commit message: configuration files corrections
added corrections to robot urdf files (my_robot.xacro, my_robot.gazebo and mapping.launch files. most of them are documented on Q&A section of udacity.

File: catkin_ws/src/my_robot/urdf/my_robot.xacro (robot description, xacro)
@@ -181,5 +181,5 @@
   <joint name="camera_optical_joint" type="fixed">
     <origin xyz="0 0 0" rpy="-1.5707 0 -1.5707"/>
-    <parent link="camera_link"/>
+    <parent link="camera"/>
     <child link="camera_link_optical"/>
   </joint>
